File: spincoater-v1/spincoater-v1.kicad_pcb (KiCad board)
At the start: 2 copper layers, 146 x 140.5 mm, 36 parts, among them J1 KEYPAD, J2 POT_PIN28, J3 SDCARD, J4 POT_PIN27, J5 MOTOR, J6 LED1, J7 LED2, J8 12V_DC, J9 LCD, Q1 IRF9540N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

Commit message: fixed trace issue
Connections:
- RV1 pad 1: +3.3V -> GND
- RV2 pad 3: +3.3V -> GND
Changed lines of the file:
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@@
 			(layers "*.Cu" "*.Mask")
 			(remove_unused_layers no)
-			(net 15 "+3.3V")
+			(net 2 "GND")
 			(pinfunction "3")
 			(pintype "passive")
@@
 			(layers "*.Cu" "*.Mask")
 			(remove_unused_layers no)
-			(net 15 "+3.3V")
+			(net 2 "GND")
 			(pinfunction "1")
 			(pintype "passive")

Commit message: added silkscreen, fixed RPi Pico position on PCB.
Other:
- board size 146 x 140.5 mm -> 141 x 140.5 mm
- board text added: "12V"
- board text added: "FUSE"
- board text added: "GND"
- board text added: "KEYPAD"
- board text added: "LCD"
- board text added: "LCD Brightness"
- board text added: "LCD Contrast"
- board text added: "MOTOR"
- board text added: "POT_PIN27"
- board text added: "POT_PIN28"
- board text added: "RPi Pico"
- board text added: "SD CARD"
Changed lines of the file:
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@@
 		)
 		(property "Value" "POT_PIN27"
-			(at 2.975 2.525 180)
+			(at -3.2831 8.84 180)
 			(layer "F.Fab")
 			(effects
@@
 		)
 		(property "Value" "POT_PIN28"
-			(at 2.92 2.5 180)
+			(at -2.8081 -6.175 180)
 			(layer "F.Fab")
 			(effects
@@
 		)
 		(property "Value" "12V_DC"
-			(at 2.7169 0.975 180)
+			(at 0.2169 7.475 180)
 			(layer "F.Fab")
 			(effects
@@
 		)
 		(property "Value" "MOTOR"
-			(at 3 4.04 180)
+			(at -2.7831 3.75 180)
 			(layer "F.Fab")
 			(effects
@@
 	)
 	(gr_circle
-		(center 61 153.5)
-		(end 63 153.5)
+		(center 65.5 153.5)
+		(end 67.5 153.5)
 		(stroke
 			(width 0.05)
@@
 	)
 	(gr_rect
-		(start 56 17.5)
+		(start 61 17.5)
 		(end 202 158)
 		(stroke
@@
 	)
 	(gr_circle
-		(center 61 22.5)
-		(end 63 22.5)
+		(center 65.5 22.5)
+		(end 67.5 22.5)
 		(stroke
 			(width 0.05)
@@
 		(layer "Edge.Cuts")
 	)
+	(gr_text "LCD Contrast"
+		(at 83.5 37 90)
+		(layer "F.SilkS")
+		(effects
+			(font
+				(size 1 1)
+				(thickness 0.1)
+			)
+			(justify left bottom)
+		)
+	)
+	(gr_text "KEYPAD"
+		(at 126.5 154.5 0)
+		(layer "F.SilkS")
+		(effects
+			(font
+				(size 1 1)
+				(thickness 0.1)
+			)
+			(justify left bottom)
+		)
+	)
+	(gr_text "12V"
+		(at 189.5 30.5 0)
+		(layer "F.SilkS")
+		(effects
+			(font
+				(size 1 1)
+				(thickness 0.1)
+			)
+			(justify left bottom)
+		)
+	)
+	(gr_text "GND"
+		(at 186 30.5 0)
+		(layer "F.SilkS")
+		(effects
+			(font
+				(size 1 1)
+				(thickness 0.1)
+			)
+			(justify left bottom)
+		)
+	)
+	(gr_text "LCD Brightness"
+		(at 65 37.5 90)
+		(layer "F.SilkS")
+		(effects
+			(font
+				(size 1 1)
+				(thickness 0.1)
+			)
+			(justify left bottom)
+		)
+	)
+	(gr_text "LCD"
+		(at 114.5 39 0)
+		(layer "F.SilkS")
+		(effects
+			(font
+				(size 1 1)
+				(thickness 0.1)
+			)
+			(justify left bottom)
+		)
+	)
+	(gr_text "RPi Pico"
+		(at 74 122 0)
+		(layer "F.SilkS")
+		(effects
+			(font
+				(size 1 1)
+				(thickness 0.1)
+			)
+			(justify left bottom)
+		)
+	)
+	(gr_text "FUSE"
+		(at 197.5 116.5 90)
+		(layer "F.SilkS")
+		(effects
+			(font
+				(size 1 1)
+				(thickness 0.1)
+			)
+			(justify left bottom)
+		)
+	)
+	(gr_text "POT_PIN28"
+		(at 152.5 140.5 0)
+		(layer "F.SilkS")
+		(effects
+			(font
+				(size 1 1)
+				(thickness 0.1)
+			)
+			(justify left bottom)
+		)
+	)
+	(gr_text "MOTOR"
+		(at 126.5 25 0)
+		(layer "F.SilkS")
+		(effects
+			(font
+				(size 1 1)
+				(thickness 0.1)
+			)
+			(justify left bottom)
+		)
+	)
+	(gr_text "POT_PIN27"
+		(at 169.5 140.5 0)
+		(layer "F.SilkS")
+		(effects
+			(font
+				(size 1 1)
+				(thickness 0.1)
+			)
+			(justify left bottom)
+		)
+	)
+	(gr_text "SD CARD"
+		(at 62 93 -90)
+		(layer "F.SilkS")
+		(effects
+			(font
+				(size 1 1)
+				(thickness 0.1)
+			)
+			(justify left bottom)
+		)
+	)
 	(segment
