File: spincoater-v1/Spincoater V2 KiCad/spincoater-v2.kicad_pcb (KiCad board)
At the start: 2 copper layers, 105 x 80 mm, 36 parts, among them J1 KEYPAD, J2 POT_PIN28, J3 SDCARD, J4 POT_PIN27, J5 MOTOR, J6 LED1, J7 LED2, J8 12V_DC, J9 LCD, Q1 IRF9540N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

Commit message: Created rough layout for new version of PCB. Fits in required space.
Parts:
- Q1, U3: footprint Package_TO_SOT_THT:TO-220-3_Horizontal_TabUp -> Package_TO_SOT_THT:TO-220-3_Vertical
- Q2, Q3: footprint Package_TO_SOT_THT:TO-92_Inline_Horizontal1 -> Package_TO_SOT_THT:TO-92_Inline
- moved J8 99.9 mm to (150.0, 32.0)
- moved Q3 98.8 mm to (136.2, 51.4)
- moved F1 96.8 mm to (163.0, 90.2)
- moved Q2 87.9 mm to (128.7, 51.4)
- moved U3 85.6 mm to (148.5, 65.0)
- moved D6 85.6 mm to (146.0, 56.2)
- moved C5 85.4 mm to (151.4, 49.5)
- moved C6 85.4 mm to (151.4, 51.5)
- moved R3 85.1 mm to (132.9, 39.0)
- moved D3 85.1 mm to (127.9, 44.5)
- moved C4 85.1 mm to (151.3, 37.5)
- moved D4 85.1 mm to (146.2, 44.5)
- moved R4 85.1 mm to (151.2, 39.5)
- moved Q1 84.7 mm to (131.4, 65.0)
- moved R2 83.5 mm to (133.9, 57.0)
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