File: Piezo-Nanopositioner-V1/PCB Design/V1/piezo_nanopositioner_v1/Z_DAC.kicad_sch (KiCad schematic)
At the start: 29 parts, among them J8 Conn_01x10_Pin, J9 RF2-04A-T-00-50-G, U10 TL431AIDBZR, U11 DAC0800LCM, U12 TDA2050

Commit message: started PCB design, almost finished first DAC.
Parts:
- removed J9: RF2-04A-T-00-50-G, RF:CONN_RF2-04A-T-00-50-G_ADM, symbol SMA_Connector:RF2-04A-T-00-50-G
- added J2: RF2-04A-T-00-50-G, CONN_RF2-04A-T-00-50-G_ADM, symbol SMA_Connector:RF2-04A-T-00-50-G
Connections:
- net at C39.2, R51.2, R52.1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: now also J2.1 (Sig)
Changed lines of the file:
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@@
+	(wire
+		(pts
+			(xy 217.17 106.68) (xy 224.79 106.68)
+		)
+		(stroke
+			(width 0)
+			(type default)
+		)
+	)
 	(wire
 		(pts
@@
 		(pts
 			(xy 138.43 135.89) (xy 146.05 135.89)
-		)
-		(stroke
-			(width 0)
-			(type default)
-		)
-	)
-	(wire
-		(pts
-			(xy 217.17 106.68) (xy 224.79 106.68)
 		)
 		(stroke
@@
 	)
 	(symbol
-		(lib_id "SMA_Connector:RF2-04A-T-00-50-G")
-		(at 224.79 106.68 0)
-		(unit 1)
-		(exclude_from_sim no)
-		(in_bom yes)
-		(on_board yes)
-		(dnp no)
-		(fields_autoplaced yes)
-		(property "Reference" "J9"
-			(at 238.76 105.4099 0)
-			(effects
-				(font
-					(size 1.524 1.524)
-				)
-				(justify left)
-			)
-		)
-		(property "Value" "RF2-04A-T-00-50-G"
-			(at 238.76 107.9499 0)
-			(effects
-				(font
-					(size 1.524 1.524)
-				)
-				(justify left)
-			)
-		)
-		(property "Footprint" "RF:CONN_RF2-04A-T-00-50-G_ADM"
-			(at 224.79 106.68 0)
-			(effects
-				(font
-					(size 1.27 1.27)
-					(italic yes)
-				)
-				(hide yes)
-			)
-		)
-		(property "Datasheet" "RF2-04A-T-00-50-G"
-			(at 224.79 106.68 0)
-			(effects
-				(font
-					(size 1.27 1.27)
-					(italic yes)
-				)
-				(hide yes)
-			)
-		)
-		(property "Description" ""
-			(at 224.79 106.68 0)
-			(effects
-				(font
-					(size 1.27 1.27)
-				)
-				(hide yes)
-			)
-		)
-		(pin "1"
-		)
-		(instances
-			(project "piezo_nanopositioner_v1"
-				(path "/7b2a32d8-cc7d-471d-a8eb-eea62713ed45/1b533877-0759-4ff4-afbe-7d3193837966"
-					(reference "J9")
-					(unit 1)
-				)
-			)
-		)
-	)
-	(symbol
 		(lib_id "Device:C")
 		(at 204.47 125.73 0)
@@
 					(unit 1)
 				)
+			)
+		)
+	)
+	(symbol
+		(lib_id "SMA_Connector:RF2-04A-T-00-50-G")
+		(at 224.79 106.68 0)
+		(unit 1)
+		(exclude_from_sim no)
+		(in_bom yes)
+		(on_board yes)
+		(dnp no)
+		(fields_autoplaced yes)
+		(property "Reference" "J2"
+			(at 238.76 105.4099 0)
+			(effects
+				(font
+					(size 1.524 1.524)
+				)
+				(justify left)
+			)
+		)
+		(property "Value" "RF2-04A-T-00-50-G"
+			(at 238.76 107.9499 0)
+			(effects
+				(font
+					(size 1.524 1.524)
+				)
+				(justify left)
+			)
+		)
+		(property "Footprint" "CONN_RF2-04A-T-00-50-G_ADM"
+			(at 225.552 97.536 0)
+			(effects
+				(font
+					(size 1.27 1.27)
+					(italic yes)
+				)
+				(hide yes)
+			)
+		)
+		(property "Datasheet" "RF2-04A-T-00-50-G"
+			(at 217.17 109.474 0)
+			(effects
+				(font
+					(size 1.27 1.27)
+					(italic yes)
+				)
+				(hide yes)
+			)
+		)
+		(property "Description" ""
+			(at 224.79 106.68 0)
+			(effects
+				(font
+					(size 1.27 1.27)
+				)
+				(hide yes)
+			)
+		)
+		(pin "1"
+		)
+		(instances
+			(project ""
+				(path "/7b2a32d8-cc7d-471d-a8eb-eea62713ed45/1b533877-0759-4ff4-afbe-7d3193837966"
+					(reference "J2")
+					(unit 1)
+				)

Commit message: Created rough PCB component layout for Z actuator.
Parts:
- renumbered C33 to C401, C34 to C402, C35 to C403, C36 to C404, C37 to C405, C38 to C406, C39 to C407, C40 to C408, C41 to C409, C42 to C410, J8 to J401, J2 to J402, R40 to R401, R41 to R402, R42 to R403, R43 to R404, R44 to R405, R45 to R406, R46 to R407, R47 to R408, R48 to R409, R49 to R410, R50 to R411, R51 to R412, R52 to R413, RV4 to RV401, U10 to U401, U11 to U402, U12 to U403
